Commit message: Update structures of xacro

File: rtk_gps_description/urdf/adl200_description.urdf.xacro (robot description, xacro)
@@ -1,10 +1,11 @@
 <?xml version="1.0"?>
 <robot xmlns:xacro="http://www.ros.org/wiki/xacro" name="robot">
+  <xacro:include filename="$(find rtk_gps_description)/urdf/materials.xacro"/>
   <xacro:include filename="$(find rtk_gps_description)/urdf/robot_core.xacro"/>
   <xacro:include filename="$(find rtk_gps_description)/urdf/sensor.xacro"/>
   <xacro:include filename="$(find rtk_gps_description)/urdf/wheel_macro.xacro"/>
-  <xacro:include filename="gps.xacro"/>
-  <xacro:include filename="gps2.xacro"/>
-  <xacro:include filename = "imu.xacro"/>
+  <xacro:include filename="$(find rtk_gps_description)/urdf/gps.xacro"/>
+  <xacro:include filename="$(find rtk_gps_description)/urdf/gps2.xacro"/>
+  <xacro:include filename="$(find rtk_gps_description)/urdf/imu.xacro"/>
   <!--xacro:include filename="$(find rtk_gps_description)/urdf/gazebo_control.xacro"/-->
   <xacro:include filename="$(find rtk_gps_description)/urdf/gazebo_controller_skid.xacro"/>

File: rtk_gps_description/urdf/gps2.xacro (robot description, xacro)
@@ -1,25 +1,25 @@
 <?xml version="1.0"?>
 <robot name="sensor_gps" xmlns:xacro="http://www.ros.org/wiki/xacro">
-        <gazebo>
-            <plugin name="gazebo_ros_gps" filename="libhector_gazebo_ros_gps.so">
-                <updateRate>4</updateRate>
-                <bodyName>sensor</bodyName>
-                <frameId>sensor</frameId>
-                <topicName>/rtk</topicName>
-                <velocityTopicName>/rtkvelocity</velocityTopicName>
-                <referenceLatitude>37.373669</referenceLatitude>
-                <referenceLongitude>126.667134</referenceLongitude>
-                <referenceHeading>90</referenceHeading>
-                <referenceAltitude>0</referenceAltitude>
-                <offset>0 0 0</offset>
-                <drift>0 0 0</drift>
-                <gaussianNoise>0 0 0</gaussianNoise>
-                <velocityDrift>0 0 0</velocityDrift>
-                <velocityGaussianNoise>0 0 0</velocityGaussianNoise>
+    <gazebo>
+        <plugin name="gazebo_ros_gps" filename="libhector_gazebo_ros_gps.so">
+            <updateRate>4</updateRate>
+            <bodyName>sensor</bodyName>
+            <frameId>sensor</frameId>
+            <topicName>/rtk</topicName>
+            <velocityTopicName>/rtkvelocity</velocityTopicName>
+            <referenceLatitude>37.373669</referenceLatitude>
+            <referenceLongitude>126.667134</referenceLongitude>
+            <referenceHeading>90</referenceHeading>
+            <referenceAltitude>0</referenceAltitude>
+            <offset>0 0 0</offset>
+            <drift>0 0 0</drift>
+            <gaussianNoise>0 0 0</gaussianNoise>
+            <velocityDrift>0 0 0</velocityDrift>
+            <velocityGaussianNoise>0 0 0</velocityGaussianNoise>
 <!--                <drift>0.001 0.001 0.001</drift>-->
 <!--                <gaussianNoise>0.05 0.05 0.05</gaussianNoise>-->
 <!--                <velocityDrift>0.001 0.001 0.001</velocityDrift>-->
 <!--                <velocityGaussianNoise>0.05 0.05 0.05</velocityGaussianNoise>-->
-            </plugin>
-        </gazebo>
+        </plugin>
+    </gazebo>
 </robot>

File: rtk_gps_description/urdf/imu.xacro (robot description, xacro)
@@ -1,5 +1,4 @@
 <?xml version="1.0"?>
 <robot name="sensor_imu" xmlns:xacro="http://www.ros.org/wiki/xacro">
-<!-- camera -->
   <gazebo>
     <!--plugin name="imu_plugin" filename="libgazebo_ros_imu.so"-->
@@ -8,8 +7,8 @@
       <boyName>sensor</boyName>
       <topicName>/handsfree/imu</topicName>
-     <frameId>sensor</frameId>
-     <accelGaussianNoise>0 0 0</accelGaussianNoise>
-     <rateGaussianNoise>0 0 0</rateGaussianNoise>
-     <yawGaussianNoise>0.0</yawGaussianNoise>
+      <frameId>sensor</frameId>
+      <accelGaussianNoise>0 0 0</accelGaussianNoise>
+      <rateGaussianNoise>0 0 0</rateGaussianNoise>
+      <yawGaussianNoise>0.0</yawGaussianNoise>
       <!--alwaysOn>true</alwaysOn>
       <bodyName>sensor</bodyName>

File: rtk_gps_description/urdf/robot_core.xacro (robot description, xacro)
@@ -1,16 +1,4 @@
 <?xml version="1.0"?>
 <robot xmlns:xacro="http://www.ros.org/wiki/xacro" >
-    <material name="white">
-        <color rgba="1 1 1 1"/>
-    </material>
-    <material name="orange">
-        <color rgba="1 0.3 0.1 1"/>
-    </material>
-    <material name="blue">
-        <color rgba="0.2 0.2 1 1"/>
-    </material>
-    <material name="black">
-        <color rgba="0 0 0 1"/>
-    </material>
     <!--BASE LINK-->
     <link name="base_link">

File: rtk_gps_description/urdf/sensor.xacro (robot description, xacro)
@@ -34,5 +34,5 @@
     </inertial>
   </link>
- <gazebo reference="sensor">
+  <gazebo reference="sensor">
     <material>Gazebo/Orange</material>
   </gazebo>
