Commit message: Permitir ingreso de xacro, antes solo urdf

File: rtk_gps_description/urdf/robot_core.xacro (robot description, xacro)
@@ -14,5 +14,5 @@
             <origin xyz= "0 0 0.085"/>
             <geometry>
-                <mesh filename= "file:///home/ros2iesus/ros2_ws/src/car_gps/rtk_gps_description/meshes/Chassis.stl" scale="0.001 0.001 0.001"/>
+                <mesh filename= "file:///home/rov-robot/colcon_ws/src/car_gps/rtk_gps_description/meshes/Chassis.stl" scale="0.001 0.001 0.001"/>
             </geometry>
             <material name ="white"/>

File: rtk_gps_description/urdf/wheel_macro.xacro (robot description, xacro)
@@ -11,5 +11,5 @@
             <visual>
                 <geometry>
-                    <mesh filename="file:///home/ros2iesus/ros2_ws/src/car_gps/rtk_gps_description/meshes/wheels.stl" scale="0.001 0.001 0.001"/>
+                    <mesh filename="file:///home/rov-robot/colcon_ws/src/car_gps/rtk_gps_description/meshes/wheels.stl" scale="0.001 0.001 0.001"/>
                 </geometry>
                 <material name="black"/>
