Commit message: Mejora de los frames del robot

File: rtk_gps_description/urdf/gazebo_controller_skid.xacro (robot description, xacro)
@@ -23,5 +23,5 @@
       <odometry_topic>odom</odometry_topic>
       <odometry_frame>odom</odometry_frame>
-      <robot_base_frame>base_link</robot_base_frame>
+      <robot_base_frame>base_footprint</robot_base_frame>
       <publish_odom>true</publish_odom>
       <publish_odom_tf>true</publish_odom_tf>

File: rtk_gps_description/urdf/robot_core.xacro (robot description, xacro)
@@ -2,13 +2,13 @@
 <robot xmlns:xacro="http://www.ros.org/wiki/xacro" >
     <!--BASE LINK-->
-    <link name="base_link">
+    <link name="base_footprint">
     </link>
     <!--CHASSIS LINK-->
-    <joint name="chassis_joint" type="fixed">
-        <parent link = "base_link"/>
-        <child link = "chassis"/>
+    <joint name="base_joint" type="fixed">
+        <parent link = "base_footprint"/>
+        <child link = "base_link"/>
         <origin xyz = "0 0 0"/>
     </joint>
-    <link name = "chassis">
+    <link name = "base_link">
         <visual>
             <origin xyz= "0 0 0.085"/>
@@ -32,5 +32,5 @@
         </inertial>
     </link>
-    <gazebo reference = "chassis">
+    <gazebo reference = "base_link">
         <material>
             Gazebo/White
