Commit message: Cambio de color de las ruedas

File: rtk_gps_description/urdf/wheel_macro.xacro (robot description, xacro)
@@ -28,5 +28,5 @@
         </link>
         <gazebo reference="${prefix}_link">
-            <material>Gazebo/Black</material>
+            <material>Gazebo/Gray</material>
             <mu1 value="0.35"/>
             <mu2 value="0.35"/>
